Commit message: verfication of different robots

File: examples/robot_descriptions/scara/scara_control.urdf (robot description, URDF)
Before this commit: robot scara_control, 4 links, 3 joints
Links:
- link base_link: geometry collision mesh filename=scara_meshes/base_link.STL scale=5 5 5; visual mesh filename=scara_meshes/base_link.STL scale=5 5 5
- link link_1: geometry collision mesh filename=scara_meshes/link_1.STL scale=5 5 5; visual mesh filename=scara_meshes/link_1.STL scale=5 5 5
- link link_2: geometry collision mesh filename=scara_meshes/link_2.STL scale=5 5 5; visual mesh filename=scara_meshes/link_2.STL scale=5 5 5
- link link_3: geometry collision mesh filename=scara_meshes/link_3.STL scale=5 5 5; visual mesh filename=scara_meshes/link_3.STL scale=5 5 5
Joints:
- joint joint_1: origin xyz=0.065 0 0 rpy=0 0 0 -> xyz=0.325 0 0 rpy=0 0 0
- joint joint_2: origin xyz=0.028115 -0.16259 0.2335 rpy=0 0 0 -> xyz=0.140575 -0.81295 1.1675 rpy=0 0 0
- joint joint_3: limit lower=-0.08 upper=0 effort=50 velocity=1 -> lower=-0.4 upper=0 effort=50 velocity=1; origin xyz=0.10838 -0.062931 0.0386 rpy=0 0 0 -> xyz=0.5419 -0.314655 0.193 rpy=0 0 0
